File: EagleGit/IP terarko/SilovaCastV2.brd (EAGLE design)
At the start: 143.5 x 93.7 mm, 57 parts, among them Q1 BC557C, T1 BT138-V, T2 BT138-V, T3 BT138-V, T4 BT138-V

Commit message: Uprava konektoru u DPS "silova cast"
Parts:
- added CON2: (no value), con-harting:CON06
- CON1: device con-harting:CON16 -> con-harting:CON10
- moved CON1 16.7 mm to (6.35, 44.5)
- moved X1 6.35 mm to (135.9, 52.1)
- moved R16 4.58 mm to (7.62, 66.0), turned to 90 degrees
- moved LED1 3.81 mm to (7.62, 77.5)
Connections:
- removed net N$35: LED1.A, R16.1
- new net N$23: CON1.1, R5.2
- net GND: now also CON2.2, CON2.4, CON2.6; no longer CON1.1, CON1.12, CON1.14, CON1.16
- net N$17: now also CON2.5; no longer CON1.3
- net N$22: now also CON2.3; no longer CON1.5
- net N$28: now also CON1.3, R6.2; no longer CON1.7, R5.2
- net N$29: now also CON1.5, R7.2; no longer CON1.9, R6.2
- net N$30: now also CON1.7, R8.2; no longer CON1.11, R7.2
- net N$31: now also CON1.9, R16.1; no longer CON1.13, R8.2
- net N$34: now also LED1.A; no longer CON1.15
Routing:
- net N$31: track 50.5 -> 10.2 mm
- net N$34: track 26.7 -> 3.81 mm
- net N$23: track 0.00 -> 18.0 mm
- net GND: track 180.0 -> 169.8 mm
- net N$22: track 39.7 -> 49.2 mm
- net N$8: track 86.4 -> 78.5 mm
- net N$16: track 28.6 -> 22.2 mm
- net N$35: track 6.35 -> 0.00 mm
- net N_PEN: track 98.6 -> 92.3 mm
- net N$2: track 73.4 -> 76.5 mm
- net N$3: track 78.5 -> 75.8 mm
- net N$1: track 75.8 -> 73.2 mm
- net N$30: track 38.0 -> 36.0 mm
- net N$28: track 13.0 -> 11.0 mm
- net N$17: track 10.2 -> 10.8 mm
