File: EagleGit/pulsniMereniDiod/pripravekV2.sch (EAGLE design)
At the start: 21 parts, among them T1 BD240C, X1 SMKDSP_1,5/2, X2 SMKDSP_1,5/2, X3 SMKDSP_1,5/2, X4 SMKDSP_1,5/6

Commit message: VES: pripravek predelan pro vetsi rozmer rezistoru
Parts:
- added R9: 51R, rcl:R-EU_0817/22
- R1, R3, R5, R6, R7, R8: device rcl:R-EU_0411/15 -> rcl:R-EU_0817/22
- R2: value 22R -> 51R; device rcl:R-EU_0411/15 -> rcl:R-EU_0817/22
Connections:
- net EMITTER: now also R9.1
- net V+: now also R9.2
Changed lines of the file:
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@@
 </classes>
 <parts>
-<part name="R2" library="rcl" deviceset="R-EU_" device="0411/15" value="22R"/>
+<part name="R2" library="rcl" deviceset="R-EU_" device="0817/22" value="51R"/>
 <part name="D1" library="diode" deviceset="1N4004" device=""/>
 <part name="X2" library="con-phoenix-smkdsp" deviceset="SMKDSP_1,5/2" device=""/>
@@
 <part name="D4" library="diode" deviceset="1N4004" device=""/>
 <part name="R4" library="rcl" deviceset="R-EU_" device="0207/12" value="1M"/>
-<part name="R5" library="rcl" deviceset="R-EU_" device="0411/15" value="4k7"/>
-<part name="R6" library="rcl" deviceset="R-EU_" device="0411/15" value="12k"/>
+<part name="R5" library="rcl" deviceset="R-EU_" device="0817/22" value="4k7"/>
+<part name="R6" library="rcl" deviceset="R-EU_" device="0817/22" value="12k"/>
 <part name="X4" library="con-phoenix-smkdsp" deviceset="SMKDSP_1,5/6" device=""/>
-<part name="R7" library="rcl" deviceset="R-EU_" device="0411/15" value="33k"/>
-<part name="R8" library="rcl" deviceset="R-EU_" device="0411/15" value="68k"/>
+<part name="R7" library="rcl" deviceset="R-EU_" device="0817/22" value="33k"/>
+<part name="R8" library="rcl" deviceset="R-EU_" device="0817/22" value="68k"/>
 <part name="T1" library="transistor" deviceset="*-PNP-" device="TO220" value="BD240C"/>
 <part name="X1" library="con-phoenix-smkdsp" deviceset="SMKDSP_1,5/2" device=""/>
-<part name="R3" library="rcl" deviceset="R-EU_" device="0411/15" value="2k2"/>
-<part name="R1" library="rcl" deviceset="R-EU_" device="0411/15" value="820R"/>
+<part name="R3" library="rcl" deviceset="R-EU_" device="0817/22" value="2k2"/>
+<part name="R1" library="rcl" deviceset="R-EU_" device="0817/22" value="820R"/>
+<part name="R9" library="rcl" deviceset="R-EU_" device="0817/22" value="51R"/>
 </parts>
 <sheets>
@@
 <instance part="R3" gate="G$1" x="63.5" y="0" rot="R90"/>
 <instance part="R1" gate="G$1" x="63.5" y="86.36" rot="R90"/>
+<instance part="R9" gate="G$1" x="101.6" y="78.74" rot="R90"/>
 </instances>
 <busses>
@@
 <pinref part="T1" gate="G$1" pin="E"/>
 <pinref part="R2" gate="G$1" pin="1"/>
-<wire x1="91.44" y1="73.66" x2="91.44" y2="68.58" width="0.1524" layer="91"/>
+<wire x1="91.44" y1="73.66" x2="91.44" y2="71.12" width="0.1524" layer="91"/>
+<pinref part="R9" gate="G$1" pin="1"/>
+<wire x1="91.44" y1="71.12" x2="91.44" y2="68.58" width="0.1524" layer="91"/>
+<wire x1="101.6" y1="73.66" x2="101.6" y2="71.12" width="0.1524" layer="91"/>
+<wire x1="101.6" y1="71.12" x2="91.44" y2="71.12" width="0.1524" layer="91"/>
+<junction x="91.44" y="71.12"/>
 </segment>
 </net>
@@
 <junction x="55.88" y="93.98"/>
 <pinref part="R1" gate="G$1" pin="2"/>
-</segment>
-</net>
+<pinref part="R9" gate="G$1" pin="2"/>
+<wire x1="91.44" y1="93.98" x2="101.6" y2="93.98" width="0.1524" layer="91"/>
+<wire x1="101.6" y1="93.98" x2="101.6" y2="83.82" width="0.1524" layer="91"/>
+<junction x="91.44" y="93.98"/>
+</segment>
+</net>
