File: EagleGit/Termoclanky/refSpoj.brd (EAGLE design)
At the start: 114.3 x 87.3 mm, 11 parts

Commit message: Termoclanky: -finalni upravy DPS pred vyrobou
Routing:
- net N$3: track 114.7 -> 113.3 mm
- net N$7: track 120.2 -> 119.4 mm
- net N$5: track 159.3 -> 158.6 mm
Changed lines of the file:
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@@
 <layer number="45" name="Holes" color="7" fill="1" visible="no" active="yes"/>
 <layer number="46" name="Milling" color="3" fill="1" visible="no" active="yes"/>
-<layer number="47" name="Measures" color="7" fill="1" visible="no" active="yes"/>
+<layer number="47" name="Measures" color="7" fill="1" visible="yes" active="yes"/>
 <layer number="48" name="Document" color="7" fill="1" visible="yes" active="yes"/>
 <layer number="49" name="Reference" color="7" fill="1" visible="yes" active="yes"/>
@@
 <wire x1="36.83" y1="69.85" x2="44.45" y2="69.85" width="3.81" layer="16"/>
 <wire x1="44.45" y1="69.85" x2="82.55" y2="69.85" width="6.4516" layer="16"/>
-<wire x1="105.41" y1="46.99" x2="105.41" y2="58.42" width="1.27" layer="16"/>
-<wire x1="105.41" y1="58.42" x2="93.98" y2="69.85" width="1.27" layer="16"/>
-<wire x1="93.98" y1="69.85" x2="82.55" y2="69.85" width="1.27" layer="16"/>
+<wire x1="105.41" y1="46.99" x2="105.41" y2="58.42" width="1.4224" layer="16"/>
+<wire x1="105.41" y1="58.42" x2="93.98" y2="69.85" width="1.4224" layer="16"/>
+<wire x1="93.98" y1="69.85" x2="82.55" y2="69.85" width="1.4224" layer="16"/>
 </signal>
 <signal name="N$2">
@@
 <wire x1="36.83" y1="62.23" x2="44.45" y2="62.23" width="3.81" layer="16"/>
 <wire x1="44.45" y1="62.23" x2="82.55" y2="62.23" width="6.4516" layer="16"/>
-<wire x1="102.87" y1="46.99" x2="102.87" y2="57.15" width="1.27" layer="16"/>
-<wire x1="102.87" y1="57.15" x2="97.79" y2="62.23" width="1.27" layer="16"/>
-<wire x1="97.79" y1="62.23" x2="82.55" y2="62.23" width="1.27" layer="16"/>
+<wire x1="102.87" y1="46.99" x2="102.87" y2="57.15" width="1.4224" layer="16"/>
+<wire x1="102.87" y1="57.15" x2="97.79" y2="62.23" width="1.4224" layer="16"/>
+<wire x1="97.79" y1="62.23" x2="82.55" y2="62.23" width="1.4224" layer="16"/>
 </signal>
 <signal name="N$3">
@@
 <wire x1="90.17" y1="54.61" x2="110.49" y2="54.61" width="1.016" layer="1"/>
 <via x="110.49" y="54.61" extent="1-16" drill="1" diameter="1.9304"/>
-<wire x1="110.49" y1="54.61" x2="110.49" y2="44.45" width="1.27" layer="16"/>
-<wire x1="110.49" y1="44.45" x2="105.41" y2="44.45" width="1.27" layer="16"/>
 <wire x1="20.32" y1="54.61" x2="26.67" y2="54.61" width="3.81" layer="16"/>
-<wire x1="82.55" y1="54.61" x2="90.17" y2="54.61" width="1.27" layer="16"/>
+<wire x1="82.55" y1="54.61" x2="90.17" y2="54.61" width="1.4224" layer="16"/>
 <wire x1="26.67" y1="54.61" x2="36.83" y2="54.61" width="6.4516" layer="16"/>
 <wire x1="36.83" y1="54.61" x2="44.45" y2="54.61" width="3.81" layer="16"/>
 <wire x1="44.45" y1="54.61" x2="82.55" y2="54.61" width="6.4516" layer="16"/>
+<wire x1="110.49" y1="54.61" x2="110.49" y2="46.99" width="1.4224" layer="16"/>
+<wire x1="110.49" y1="46.99" x2="107.95" y2="44.45" width="1.4224" layer="16"/>
+<wire x1="107.95" y1="44.45" x2="105.41" y2="44.45" width="1.4224" layer="16"/>
 </signal>
 <signal name="N$4">
@@
 <contactref element="CON1" pad="3"/>
 <wire x1="12.7" y1="50.8" x2="16.51" y2="46.99" width="3.81" layer="16"/>
-<wire x1="102.87" y1="44.45" x2="92.71" y2="44.45" width="1.27" layer="16"/>
-<wire x1="92.71" y1="44.45" x2="90.17" y2="46.99" width="1.27" layer="16"/>
+<wire x1="102.87" y1="44.45" x2="92.71" y2="44.45" width="1.4224" layer="16"/>
+<wire x1="92.71" y1="44.45" x2="90.17" y2="46.99" width="1.4224" layer="16"/>
 <wire x1="16.51" y1="46.99" x2="26.67" y2="46.99" width="3.81" layer="16"/>
-<wire x1="82.55" y1="46.99" x2="90.17" y2="46.99" width="1.27" layer="16"/>
+<wire x1="82.55" y1="46.99" x2="90.17" y2="46.99" width="1.4224" layer="16"/>
 <wire x1="26.67" y1="46.99" x2="36.83" y2="46.99" width="6.4516" layer="16"/>
 <wire x1="36.83" y1="46.99" x2="44.45" y2="46.99" width="3.81" layer="16"/>
@@
 <wire x1="90.17" y1="39.37" x2="90.17" y2="11.43" width="1.016" layer="1"/>
 <via x="90.17" y="11.43" extent="1-16" drill="1" diameter="1.9304"/>
-<wire x1="111.76" y1="41.91" x2="105.41" y2="41.91" width="1.27" layer="16"/>
 <wire x1="16.51" y1="39.37" x2="26.67" y2="39.37" width="3.81" layer="16"/>
-<wire x1="82.55" y1="39.37" x2="90.17" y2="39.37" width="1.27" layer="16"/>
+<wire x1="82.55" y1="39.37" x2="90.17" y2="39.37" width="1.4224" layer="16"/>
 <wire x1="26.67" y1="39.37" x2="36.83" y2="39.37" width="6.4516" layer="16"/>
 <wire x1="36.83" y1="39.37" x2="44.45" y2="39.37" width="3.81" layer="16"/>
 <wire x1="44.45" y1="39.37" x2="82.55" y2="39.37" width="6.4516" layer="16"/>
-<wire x1="90.17" y1="11.43" x2="101.6" y2="11.43" width="1.27" layer="16"/>
-<wire x1="101.6" y1="11.43" x2="111.76" y2="21.59" width="1.27" layer="16"/>
-<wire x1="111.76" y1="21.59" x2="111.76" y2="41.91" width="1.27" layer="16"/>
+<wire x1="90.17" y1="11.43" x2="101.6" y2="11.43" width="1.4224" layer="16"/>
+<wire x1="101.6" y1="11.43" x2="111.76" y2="21.59" width="1.4224" layer="16"/>
+<wire x1="105.41" y1="41.91" x2="110.49" y2="41.91" width="1.4224" layer="16"/>
+<wire x1="110.49" y1="41.91" x2="111.76" y2="40.64" width="1.4224" layer="16"/>
+<wire x1="111.76" y1="40.64" x2="111.76" y2="21.59" width="1.4224" layer="16"/>
 </signal>
 <signal name="N$6">
@@
 <wire x1="12.7" y1="27.94" x2="16.51" y2="27.94" width="3.81" layer="16"/>
 <wire x1="16.51" y1="27.94" x2="20.32" y2="31.75" width="3.81" layer="16"/>
-<wire x1="99.06" y1="41.91" x2="102.87" y2="41.91" width="1.27" layer="16"/>
-<wire x1="92.71" y1="31.75" x2="93.98" y2="33.02" width="1.27" layer="16"/>
-<wire x1="93.98" y1="33.02" x2="93.98" y2="36.83" width="1.27" layer="16"/>
-<wire x1="93.98" y1="36.83" x2="99.06" y2="41.91" width="1.27" layer="16"/>
+<wire x1="99.06" y1="41.91" x2="102.87" y2="41.91" width="1.4224" layer="16"/>
+<wire x1="92.71" y1="31.75" x2="93.98" y2="33.02" width="1.4224" layer="16"/>
+<wire x1="93.98" y1="33.02" x2="93.98" y2="36.83" width="1.4224" layer="16"/>
+<wire x1="93.98" y1="36.83" x2="99.06" y2="41.91" width="1.4224" layer="16"/>
 <wire x1="20.32" y1="31.75" x2="26.67" y2="31.75" width="3.81" layer="16"/>
-<wire x1="82.55" y1="31.75" x2="92.71" y2="31.75" width="1.27" layer="16"/>
+<wire x1="82.55" y1="31.75" x2="92.71" y2="31.75" width="1.4224" layer="16"/>
 <wire x1="26.67" y1="31.75" x2="36.83" y2="31.75" width="6.4516" layer="16"/>
 <wire x1="36.83" y1="31.75" x2="44.45" y2="31.75" width="3.81" layer="16"/>
@@
 <wire x1="92.71" y1="24.13" x2="109.22" y2="24.13" width="1.016" layer="1"/>
 <via x="109.22" y="24.13" extent="1-16" drill="1" diameter="1.9304"/>
-<wire x1="109.22" y1="24.13" x2="109.22" y2="39.37" width="1.27" layer="16"/>
-<wire x1="109.22" y1="39.37" x2="105.41" y2="39.37" width="1.27" layer="16"/>
 <wire x1="24.13" y1="24.13" x2="26.67" y2="24.13" width="3.81" layer="16"/>
-<wire x1="82.55" y1="24.13" x2="92.71" y2="24.13" width="1.016" layer="16"/>
+<wire x1="82.55" y1="24.13" x2="92.71" y2="24.13" width="1.6764" layer="16"/>
 <wire x1="26.67" y1="24.13" x2="36.83" y2="24.13" width="6.4516" layer="16"/>
 <wire x1="36.83" y1="24.13" x2="44.45" y2="24.13" width="3.81" layer="16"/>
 <wire x1="44.45" y1="24.13" x2="82.55" y2="24.13" width="6.4516" layer="16"/>
+<wire x1="105.41" y1="39.37" x2="107.95" y2="39.37" width="1.4224" layer="16"/>
+<wire x1="107.95" y1="39.37" x2="109.22" y2="38.1" width="1.4224" layer="16"/>
+<wire x1="109.22" y1="38.1" x2="109.22" y2="24.13" width="1.4224" layer="16"/>
 </signal>
 <signal name="N$8">
@@
 <contactref element="CON1" pad="7"/>
 <wire x1="12.7" y1="5.08" x2="24.13" y2="16.51" width="3.81" layer="16"/>
-<wire x1="95.25" y1="16.51" x2="97.79" y2="19.05" width="1.27" layer="16"/>
-<wire x1="97.79" y1="19.05" x2="97.79" y2="36.83" width="1.27" layer="16"/>
-<wire x1="97.79" y1="36.83" x2="100.33" y2="39.37" width="1.27" layer="16"/>
-<wire x1="100.33" y1="39.37" x2="102.87" y2="39.37" width="1.27" layer="16"/>
+<wire x1="95.25" y1="16.51" x2="97.79" y2="19.05" width="1.4224" layer="16"/>
+<wire x1="97.79" y1="19.05" x2="97.79" y2="36.83" width="1.4224" layer="16"/>
+<wire x1="97.79" y1="36.83" x2="100.33" y2="39.37" width="1.4224" layer="16"/>
+<wire x1="100.33" y1="39.37" x2="102.87" y2="39.37" width="1.4224" layer="16"/>
 <wire x1="24.13" y1="16.51" x2="26.67" y2="16.51" width="3.81" layer="16"/>
-<wire x1="82.55" y1="16.51" x2="95.25" y2="16.51" width="1.27" layer="16"/>
+<wire x1="82.55" y1="16.51" x2="95.25" y2="16.51" width="1.4224" layer="16"/>
 <wire x1="26.67" y1="16.51" x2="36.83" y2="16.51" width="6.4516" layer="16"/>
 <wire x1="36.83" y1="16.51" x2="44.45" y2="16.51" width="3.81" layer="16"/>
