File: EagleGit/Termoclanky/zesilovac.brd (EAGLE design)
At the start: 247.6 x 134.3 mm, 94 parts, among them IC1 TL061P, IC2 TL061P, IC3 TL061P, IC4 TL061P, Q1 BD140, Q2 BD140, Q3 BD140, Q4 BD140, T1 BD139, T2 BD139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

Commit message: Rozdeleni vstupnich 50 ohmovych odporu k jednotlivym vstupum.
Parts:
- removed SV2: (no value), con-lstb:MA04-2
- added C13, C14, C15, C16: 100u, rcl:E5-13
- added SL5, SL6, SL7, SL8: (no value), con-amp-quick:03P
- moved R47 91.6 mm to (21.6, 30.5)
- moved R48 91.1 mm to (17.8, 30.5)
- moved R45 73.0 mm to (21.6, 61.0)
- moved R46 72.2 mm to (17.8, 61.0)
- moved R41 70.7 mm to (21.6, 100.3), turned to 180 degrees
- moved R43 66.6 mm to (21.6, 85.1), turned to 180 degrees
- moved C11 66.1 mm to (185.4, 92.7)
- moved R42 64.7 mm to (21.6, 104.1), turned to 180 degrees
- moved R44 64.5 mm to (21.6, 81.3), turned to 180 degrees
- moved C9 61.6 mm to (200.7, 92.7)
- moved C12 22.5 mm to (135.9, 92.7)
- moved C10 10.5 mm to (151.1, 92.7)
- moved R11 8.13 mm to (204.5, 6.35)
- moved R18 8.13 mm to (174.0, 6.35)
- moved R40 8.13 mm to (53.3, 6.35)
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Connections:
- removed net N$41: R41.1, R42.1, SV2.2
- new net N$47: R41.1, R42.1, SL5.1, SL5.2
- net GND: now also C13.-, C14.-, C15.+, C16.+
- net N$14: now also SL6.3; no longer SV2.3
- net N$22: now also SL7.3; no longer SV2.5
- net N$30: now also SL8.3; no longer SV2.7
- net N$42: now also SL6.1, SL6.2; no longer SV2.4
- net N$43: now also SL7.1, SL7.2; no longer SV2.6
- net N$44: now also SL8.1, SL8.2; no longer SV2.8
- net N$6: now also SL5.3; no longer SV2.1
- net VDD: now also C13.+, C14.+
- net VSS: now also C15.-, C16.-
Routing:
- net GND: track 635.3 -> 1135.6 mm
- net N$14: track 239.5 -> 309.0 mm
- net N$22: track 161.0 -> 217.3 mm
- net N$6: track 321.5 -> 359.4 mm
- net N$44: track 0.00 -> 14.0 mm
- net N$47: track 0.00 -> 13.8 mm
- net N$42: track 0.00 -> 13.8 mm
- net N$30: track 79.0 -> 89.9 mm
- net N$43: track 0.00 -> 10.2 mm
- net N$1: track 13.9 -> 20.2 mm
- net N$25: track 13.9 -> 20.2 mm
- net N$29: track 37.4 -> 43.7 mm
- net N$21: track 34.1 -> 40.5 mm
- net N$33: track 34.0 -> 40.4 mm
- net N$17: track 13.9 -> 20.2 mm
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
Commit message: Nova koncepce koncoveho zesilovace podle Papeze. Je treba dodelat totez pro ostatni vstupy.
Parts:
- added R53, R54: 220R, resistor:0207/12
- added R55, R56: 1k5, resistor:0207/12
- added R57, R58: 4R7, resistor:0207/12
- added R59: 5k, pot:LI10
- added T5: BD139, transistor-power:TO126AV
- Q1: device transistor-pnp:TO126 -> transistor-power:TO126AV
- R49: value 10k -> 1k5
- T1: device transistor:TO126 -> transistor-power:TO126AV
- moved PAD2 62.3 mm to (191.8, 129.5)
- moved PAD1 61.1 mm to (204.5, 129.5)
- moved PAD3 57.3 mm to (174.0, 129.5)
- moved C16 34.2 mm to (48.3, 124.5), turned to 90 degrees
- moved C13 33.9 mm to (108.0, 125.7), turned to 270 degrees
- moved C14 33.7 mm to (63.5, 124.5), turned to 270 degrees
- moved C10 33.2 mm to (154.9, 125.7), turned to 270 degrees
- moved C15 30.7 mm to (88.9, 123.2), turned to 90 degrees
- moved C12 29.3 mm to (138.4, 121.9), turned to 90 degrees
- moved T1 28.0 mm to (217.2, 83.8)
- moved C9 27.0 mm to (218.4, 113.0), turned to 90 degrees
- moved Q1 22.5 mm to (189.2, 83.8)
- moved C11 20.5 mm to (188.0, 113.0), turned to 270 degrees
- moved Q4 12.7 mm to (44.5, 62.2)
- moved T4 12.7 mm to (61.0, 62.2)
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Connections:
- new net N$41: Q1.B, R54.2, R56.1, R59.A, T5.E
- new net N$49: R53.1, R55.1, R59.E, T1.B, T5.C
- new net N$51: R57.1, T1.E
- new net N$52: Q1.E, R58.2
- new net N$53: R59.S, T5.B
- net N$3: now also R53.2, R54.1; no longer Q1.3, T1.3
- net N$46: now also R57.2, R58.1; no longer Q1.1, T1.1
- net VDD: now also R55.2, T1.C; no longer T1.2
- net VSS: now also Q1.C, R56.2; no longer Q1.2
Routing:
- net GND: track 1135.6 -> 1395.8 mm, vias 0 -> 3
- net VSS: track 229.5 -> 304.6 mm, vias 0 -> 1
- net N$49: track 0.00 -> 61.3 mm
- net N$52: track 0.00 -> 56.2 mm
- net N$41: track 0.00 -> 49.8 mm
- net N$46: track 61.7 -> 24.7 mm
- net N$37: track 81.9 -> 115.1 mm
- net VDD: track 184.2 -> 208.1 mm, vias 0 -> 1
- net N$38: track 137.9 -> 161.7 mm
- net N$45: track 35.6 -> 50.5 mm
- net N$48: track 35.6 -> 50.5 mm
- net N$10: track 69.7 -> 57.0 mm
- net N$51: track 0.00 -> 11.5 mm
- net N$3: track 35.6 -> 24.1 mm
- net N$53: track 0.00 -> 10.3 mm
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Other:
- board size 247.6 x 134.3 mm -> 254 x 134.3 mm

Commit message: Termoclanky: Hotovy navrh dps zesilovacu.
Parts:
- added C17, C18, C19, C20, C21, C22, C23, C24: 10n, capacitor-wima:C5B5
- added R60, R61, R67, R68, R74, R75: 4R7, resistor:0207/12
- added R62, R64, R69, R70, R76, R77: 1k5, resistor:0207/12
- added R63, R65, R71, R72, R78, R79: 220R, resistor:0207/12
- added R66, R73, R80: 5k, pot:LI10
- added T6, T7, T8: BD139, transistor-power:TO126AV
- added U$1, U$2, U$3, U$4: (no value), holes:3,2
- added U$5, U$6, U$7: (no value), holes:5,5
- Q2, Q3, Q4: device transistor-pnp:TO126 -> transistor-power:TO126AV
- R50, R51, R52: value 10k -> 1k5
- T2, T3, T4: device transistor:TO126 -> transistor-power:TO126AV
- moved T3 24.4 mm to (121.9, 83.8)
- moved T4 24.4 mm to (72.4, 83.8)
- moved T2 23.3 mm to (170.2, 83.8)
- moved Q3 21.6 mm to (94.0, 83.8)
- moved Q2 21.6 mm to (142.2, 83.8)
- moved Q4 21.6 mm to (44.5, 83.8)
- moved C10 20.8 mm to (171.4, 113.0), turned to 90 degrees
- moved C13 19.8 mm to (123.2, 113.0), turned to 90 degrees
- moved C14 15.3 mm to (73.7, 113.0), turned to 90 degrees
- moved X1 13.3 mm to (240.0, 34.3)
- moved X8 12.7 mm to (10.2, 34.3)
- moved C16 12.5 mm to (43.2, 113.0), turned to 270 degrees
- moved C3 11.5 mm to (110.5, 48.3)
- moved C15 10.9 mm to (92.7, 113.0), turned to 270 degrees
- moved SL1 10.2 mm to (218.4, 34.3)
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Connections:
- new net N$54: R67.1, T3.E
- new net N$55: Q2.E, R61.2
- new net N$56: Q3.E, R68.2
- new net N$57: R60.1, T2.E
- new net N$58: Q2.B, R62.1, R63.2, R66.A, T6.E
- new net N$59: R64.1, R65.1, R66.E, T2.B, T6.C
- new net N$60: R66.S, T6.B
- new net N$61: R69.1, R71.1, R73.E, T3.B, T7.C
- new net N$62: Q3.B, R70.1, R72.2, R73.A, T7.E
- new net N$63: R74.1, T4.E
- new net N$64: Q4.E, R75.2
- new net N$65: R73.S, T7.B
- new net N$68: R76.1, R79.1, R80.E, T4.B, T8.C
- new net N$69: Q4.B, R77.1, R78.2, R80.A, T8.E
- new net N$70: R80.S, T8.B
- net GND: now also C17.2, C18.2, C19.2, C20.2, C21.1, C22.1, C23.1, C24.1
- net N$10: now also R74.2, R75.1; no longer Q4.1, T4.1
- net N$18: now also R67.2, R68.1; no longer Q3.1, T3.1
- net N$26: now also R60.2, R61.1; no longer Q2.1, T2.1
- net N$45: now also R63.1, R65.2; no longer Q2.3, T2.3
- net N$48: now also R71.2, R72.1; no longer Q3.3, T3.3
- net N$50: now also R78.1, R79.2; no longer Q4.3, T4.3
- net VDD: now also C17.1, C18.1, C19.1, C20.1, R64.2, R69.2, R76.2, T2.C, T3.C, T4.C; no longer T2.2, T3.2, T4.2
- net VSS: now also C21.2, C22.2, C23.2, C24.2, Q2.C, Q3.C, Q4.C, R62.2, R70.2, R77.2; no longer Q2.2, Q3.2, Q4.2
Routing:
- net GND: track 1395.8 -> 2063.0 mm, vias 3 -> 12
- net VSS: track 304.6 -> 763.2 mm, vias 1 -> 0
- net VDD: track 208.1 -> 583.9 mm
- net N$30: track 89.9 -> 172.0 mm, vias 0 -> 2
- net N$22: track 217.3 -> 293.7 mm
- net N$64: track 0.00 -> 57.4 mm
- net N$56: track 0.00 -> 56.9 mm
- net N$55: track 0.00 -> 56.9 mm
- net N$59: track 0.00 -> 53.4 mm
- net N$68: track 0.00 -> 53.4 mm
- net N$61: track 0.00 -> 53.4 mm
- net N$69: track 0.00 -> 48.5 mm
- net N$62: track 0.00 -> 47.8 mm
- net N$58: track 0.00 -> 47.8 mm
- net N$26: track 78.1 -> 33.7 mm
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Other:
- board size 254 x 134.3 mm -> 250.2 x 134.3 mm

Commit message: Termistory: - predelany zakoncovaci rezistory na vetsi vykony - rozsireny cesty - finalni verze DPS
Parts:
- removed CON1: (no value), con-harting:CON10
- added R81, R82, R83, R84: 680R, resistor:0207/12
- added SV2: (no value), con-lstb:MA05-2
- added U$10, U$11, U$12, U$8, U$9: (no value), holes:3,2
- R29, R30, R31, R32, R33, R34, R35, R36: value 100R -> 27R; device resistor:0207/12 -> resistor:0411/12
- moved R36 172.0 mm to (238.8, 99.1)
- moved R34 116.6 mm to (238.8, 73.7)
- moved R32 66.0 mm to (238.8, 48.3)
- moved R30 31.7 mm to (238.8, 22.9)
- moved R40 19.0 mm to (33.0, 6.35)
- moved R38 14.0 mm to (88.9, 6.35)
- moved R39 14.0 mm to (58.4, 6.35)
- moved R37 8.89 mm to (114.3, 6.35)
- moved R25 8.89 mm to (144.8, 6.35)
- moved R11 3.81 mm to (200.7, 6.35)
- moved R18 3.81 mm to (170.2, 6.35)
- moved U$2 3.81 mm to (6.35, 132.1)
- moved U$3 3.81 mm to (243.8, 132.1)
- moved X4 3.81 mm to (240.0, 110.5)
- moved X5 3.81 mm to (10.2, 110.5)
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Connections:
- new net N$66: R30.1, R81.1, X1.1
- new net N$67: R32.1, R82.1, X2.1
- new net N$72: R33.1, R34.2
- new net N$73: R34.1, R83.1, X3.1
- net GND: now also R81.2, R82.2, R83.2, R84.2, SV2.10, SV2.2, SV2.4, SV2.6, SV2.8; no longer CON1.2, CON1.4, CON1.6, CON1.8
- net N$10: no longer R36.2
- net N$14: now also SV2.3; no longer CON1.3
- net N$18: no longer R34.2
- net N$22: now also SV2.5; no longer CON1.5
- net N$26: no longer R32.2
- net N$30: now also SV2.7; no longer CON1.7
- net N$36: now also R30.2; no longer R30.1, X1.1
- net N$37: now also R32.2; no longer R32.1, X2.1
- net N$38: now also R35.1, R36.2; no longer R33.1, R34.1, X3.1
- net N$39: now also R84.1; no longer R35.1
- net N$46: no longer R30.2
- net N$6: now also SV2.1; no longer CON1.1
Routing:
- net N$39: track 199.2 -> 38.9 mm
- net N$72: track 0.00 -> 160.1 mm
- net GND: track 2063.0 -> 2107.4 mm
- net N$38: track 152.2 -> 193.4 mm
- net N$73: track 0.00 -> 38.9 mm
- net N$66: track 0.00 -> 38.9 mm
- net N$67: track 0.00 -> 38.9 mm
- net N$25: track 24.3 -> 44.1 mm
- net N$17: track 24.3 -> 39.1 mm
- net N$37: track 119.4 -> 129.3 mm
- net N$22: track 293.7 -> 300.5 mm
- net N$9: track 23.3 -> 30.0 mm
- net N$13: track 15.3 -> 20.4 mm
- net N$40: track 15.3 -> 20.4 mm
- net N$34: track 15.3 -> 20.4 mm
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Other:
- board size 250.2 x 134.3 mm -> 250.2 x 138.1 mm

Commit message: Termoclanky: -finalni upravy DPS pred vyrobou
Routing:
- net GND: track 2107.4 -> 1536.4 mm
- added copper zone on layer 1, net GND
Changed lines of the file:
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@@
 <layer number="45" name="Holes" color="7" fill="1" visible="no" active="yes"/>
 <layer number="46" name="Milling" color="3" fill="1" visible="no" active="yes"/>
-<layer number="47" name="Measures" color="7" fill="1" visible="no" active="yes"/>
+<layer number="47" name="Measures" color="7" fill="1" visible="yes" active="yes"/>
 <layer number="48" name="Document" color="7" fill="1" visible="yes" active="yes"/>
 <layer number="49" name="Reference" color="7" fill="1" visible="yes" active="yes"/>
@@
 <param name="mtCopper" value="0.035mm 0.035mm 0.035mm 0.035mm 0.035mm 0.035mm 0.035mm 0.035mm 0.035mm 0.035mm 0.035mm 0.035mm 0.035mm 0.035mm 0.035mm 0.035mm"/>
 <param name="mtIsolate" value="1.5mm 0.15mm 0.2mm 0.15mm 0.2mm 0.15mm 0.2mm 0.15mm 0.2mm 0.15mm 0.2mm 0.15mm 0.2mm 0.15mm 0.2mm"/>
-<param name="mdWireWire" value="8mil"/>
-<param name="mdWirePad" value="8mil"/>
-<param name="mdWireVia" value="8mil"/>
-<param name="mdPadPad" value="8mil"/>
-<param name="mdPadVia" value="8mil"/>
-<param name="mdViaVia" value="8mil"/>
+<param name="mdWireWire" value="20mil"/>
+<param name="mdWirePad" value="20mil"/>
+<param name="mdWireVia" value="20mil"/>
+<param name="mdPadPad" value="20mil"/>
+<param name="mdPadVia" value="20mil"/>
+<param name="mdViaVia" value="20mil"/>
 <param name="mdSmdPad" value="8mil"/>
 <param name="mdSmdVia" value="8mil"/>
@@
 <param name="srMinRoundness" value="0mil"/>
 <param name="srMaxRoundness" value="0mil"/>
-<param name="slThermalIsolate" value="10mil"/>
-<param name="slThermalsForVias" value="0"/>
+<param name="slThermalIsolate" value="20mil"/>
+<param name="slThermalsForVias" value="1"/>
 <param name="dpMaxLengthDifference" value="10mm"/>
 <param name="dpGapFactor" value="2.5"/>
@@
 <contactref element="C11" pad="+"/>
 <contactref element="C12" pad="+"/>
-<wire x1="57.15" y1="48.26" x2="48.26" y2="48.26" width="1.016" layer="16"/>
+<wire x1="57.15" y1="48.26" x2="50.8" y2="48.26" width="1.016" layer="16"/>
+<wire x1="50.8" y1="48.26" x2="48.26" y2="48.26" width="1.016" layer="16"/>
 <wire x1="48.26" y1="48.26" x2="45.72" y2="45.72" width="1.016" layer="16"/>
 <wire x1="12.7" y1="24.13" x2="26.67" y2="10.16" width="1.4224" layer="16"/>
@@
 <contactref element="C13" pad="-"/>
 <wire x1="191.77" y1="45.72" x2="194.31" y2="48.26" width="1.016" layer="16"/>
-<wire x1="194.31" y1="48.26" x2="203.2" y2="48.26" width="1.016" layer="16"/>
+<wire x1="194.31" y1="48.26" x2="196.85" y2="48.26" width="1.016" layer="16"/>
 <via x="223.52" y="55.88" extent="1-16" drill="1" diameter="2.1844"/>
-<wire x1="223.52" y1="55.88" x2="189.23" y2="55.88" width="1.6764" layer="1"/>
-<via x="189.23" y="55.88" extent="1-16" drill="1" diameter="2.1844"/>
-<wire x1="189.23" y1="55.88" x2="189.23" y2="48.26" width="1.016" layer="16"/>
-<wire x1="189.23" y1="48.26" x2="191.77" y2="45.72" width="1.016" layer="16"/>
-<wire x1="189.23" y1="55.88" x2="189.23" y2="35.56" width="1.6764" layer="1"/>
-<wire x1="189.23" y1="35.56" x2="190.5" y2="34.29" width="1.6764" layer="1"/>
-<wire x1="190.5" y1="34.29" x2="190.5" y2="26.67" width="1.6764" layer="1"/>
-<wire x1="189.23" y1="55.88" x2="189.23" y2="64.77" width="1.6764" layer="1"/>
+<wire x1="196.85" y1="48.26" x2="203.2" y2="48.26" width="1.016" layer="16"/>
 <via x="203.2" y="115.57" extent="1-16" drill="1" diameter="2.1844"/>
-<wire x1="203.2" y1="115.57" x2="203.2" y2="91.44" width="1.6764" layer="1"/>
-<wire x1="203.2" y1="91.44" x2="196.85" y2="85.09" width="1.6764" layer="1"/>
-<wire x1="196.85" y1="85.09" x2="196.85" y2="72.39" width="1.6764" layer="1"/>
-<wire x1="196.85" y1="72.39" x2="189.23" y2="64.77" width="1.6764" layer="1"/>
 <wire x1="226.06" y1="93.98" x2="187.96" y2="93.98" width="1.4224" layer="16"/>
-<wire x1="156.21" y1="48.26" x2="147.32" y2="48.26" width="1.016" layer="16"/>
+<wire x1="156.21" y1="48.26" x2="149.86" y2="48.26" width="1.016" layer="16"/>
+<wire x1="149.86" y1="48.26" x2="147.32" y2="48.26" width="1.016" layer="16"/>
 <wire x1="147.32" y1="48.26" x2="144.78" y2="45.72" width="1.016" layer="16"/>
 <via x="176.53" y="55.88" extent="1-16" drill="1" diameter="2.1844"/>
-<wire x1="176.53" y1="55.88" x2="142.24" y2="55.88" width="1.6764" layer="1"/>
-<via x="142.24" y="55.88" extent="1-16" drill="1" diameter="2.1844"/>
-<wire x1="142.24" y1="55.88" x2="142.24" y2="48.26" width="1.016" layer="16"/>
-<wire x1="142.24" y1="48.26" x2="144.78" y2="45.72" width="1.016" layer="16"/>
 <via x="156.21" y="115.57" extent="1-16" drill="1" diameter="2.1844"/>
-<wire x1="156.21" y1="115.57" x2="156.21" y2="91.44" width="1.6764" layer="1"/>
-<wire x1="156.21" y1="91.44" x2="149.86" y2="85.09" width="1.6764" layer="1"/>
-<wire x1="149.86" y1="85.09" x2="149.86" y2="72.39" width="1.6764" layer="1"/>
-<wire x1="149.86" y1="72.39" x2="142.24" y2="64.77" width="1.6764" layer="1"/>
-<wire x1="142.24" y1="64.77" x2="142.24" y2="55.88" width="1.6764" layer="1"/>
 <wire x1="187.96" y1="115.57" x2="171.45" y2="115.57" width="1.6764" layer="16"/>
-<wire x1="143.51" y1="26.67" x2="143.51" y2="34.29" width="1.6764" layer="1"/>
-<wire x1="143.51" y1="34.29" x2="142.24" y2="35.56" width="1.6764" layer="1"/>
-<wire x1="142.24" y1="35.56" x2="142.24" y2="55.88" width="1.6764" layer="1"/>
-<wire x1="107.95" y1="48.26" x2="99.06" y2="48.26" width="1.016" layer="16"/>
+<wire x1="107.95" y1="48.26" x2="101.6" y2="48.26" width="1.016" layer="16"/>
+<wire x1="101.6" y1="48.26" x2="99.06" y2="48.26" width="1.016" layer="16"/>
 <wire x1="99.06" y1="48.26" x2="96.52" y2="45.72" width="1.016" layer="16"/>
 <via x="107.95" y="115.57" extent="1-16" drill="1" diameter="2.1844"/>
-<wire x1="107.95" y1="115.57" x2="107.95" y2="92.71" width="1.6764" layer="1"/>
-<wire x1="107.95" y1="92.71" x2="101.6" y2="86.36" width="1.6764" layer="1"/>
-<wire x1="101.6" y1="86.36" x2="101.6" y2="72.39" width="1.6764" layer="1"/>
-<wire x1="101.6" y1="72.39" x2="93.98" y2="64.77" width="1.6764" layer="1"/>
-<wire x1="93.98" y1="64.77" x2="93.98" y2="55.88" width="1.6764" layer="1"/>
-<via x="93.98" y="55.88" extent="1-16" drill="1" diameter="2.1844"/>
-<wire x1="93.98" y1="55.88" x2="93.98" y2="48.26" width="1.016" layer="16"/>
-<wire x1="93.98" y1="48.26" x2="96.52" y2="45.72" width="1.016" layer="16"/>
 <wire x1="123.19" y1="115.57" x2="140.97" y2="115.57" width="1.6764" layer="16"/>
 <wire x1="228.6" y1="99.06" x2="146.05" y2="99.06" width="1.4224" layer="16"/>
 <via x="128.27" y="55.88" extent="1-16" drill="1" diameter="2.1844"/>
-<wire x1="128.27" y1="55.88" x2="93.98" y2="55.88" width="1.6764" layer="1"/>
-<wire x1="95.25" y1="26.67" x2="95.25" y2="34.29" width="1.6764" layer="1"/>
-<wire x1="95.25" y1="34.29" x2="93.98" y2="35.56" width="1.6764" layer="1"/>
-<wire x1="93.98" y1="35.56" x2="93.98" y2="55.88" width="1.6764" layer="1"/>
 <wire x1="25.4" y1="48.26" x2="26.67" y2="48.26" width="1.4224" layer="16"/>
 <wire x1="74.93" y1="53.34" x2="74.93" y2="35.56" width="1.4224" layer="16"/>
@@
 <wire x1="86.36" y1="57.15" x2="85.09" y2="55.88" width="1.4224" layer="16"/>
 <via x="85.09" y="55.88" extent="1-16" drill="1" diameter="2.1844"/>
-<wire x1="85.09" y1="55.88" x2="43.18" y2="55.88" width="1.6764" layer="1"/>
-<via x="43.18" y="55.88" extent="1-16" drill="1" diameter="2.1844"/>
-<wire x1="43.18" y1="55.88" x2="43.18" y2="48.26" width="1.016" layer="16"/>
-<wire x1="43.18" y1="48.26" x2="45.72" y2="45.72" width="1.016" layer="16"/>
-<wire x1="44.45" y1="26.67" x2="44.45" y2="34.29" width="1.6764" layer="1"/>
-<wire x1="44.45" y1="34.29" x2="43.18" y2="35.56" width="1.6764" layer="1"/>
-<wire x1="43.18" y1="35.56" x2="43.18" y2="55.88" width="1.6764" layer="1"/>
 <via x="58.42" y="115.57" extent="1-16" drill="1" diameter="2.1844"/>
-<wire x1="58.42" y1="115.57" x2="58.42" y2="92.71" width="1.6764" layer="1"/>
-<wire x1="58.42" y1="92.71" x2="52.07" y2="86.36" width="1.6764" layer="1"/>
-<wire x1="52.07" y1="86.36" x2="52.07" y2="73.66" width="1.6764" layer="1"/>
-<wire x1="52.07" y1="73.66" x2="43.18" y2="64.77" width="1.6764" layer="1"/>
-<wire x1="43.18" y1="64.77" x2="43.18" y2="55.88" width="1.6764" layer="1"/>
 <wire x1="25.4" y1="24.13" x2="41.91" y2="24.13" width="1.4224" layer="16"/>
 <wire x1="41.91" y1="24.13" x2="44.45" y2="26.67" width="1.4224" layer="16"/>
@@
 <wire x1="38.1" y1="133.35" x2="36.83" y2="134.62" width="1.4224" layer="16"/>
 <wire x1="36.83" y1="134.62" x2="35.56" y2="134.62" width="1.4224" layer="16"/>
+<polygon width="0.4064" layer="1">
+<vertex x="35.56" y="120.65"/>
+<vertex x="228.6" y="120.65"/>
+<vertex x="228.6" y="16.51"/>
+<vertex x="30.48" y="16.51"/>
+<vertex x="30.48" y="42.545"/>
+<vertex x="35.56" y="47.625"/>
+</polygon>
+<via x="50.8" y="48.26" extent="1-16" drill="1" diameter="2.1844"/>
+<via x="101.6" y="48.26" extent="1-16" drill="1" diameter="2.1844"/>
+<via x="149.86" y="48.26" extent="1-16" drill="1" diameter="2.1844"/>
+<via x="196.85" y="48.26" extent="1-16" drill="1" diameter="2.1844"/>
 </signal>
 <signal name="N$1">
