File: EagleGit/quanti/ICM20600-pan.brd (EAGLE design)
At the start: 35.5 x 30.1 mm, 21 parts, among them IC1 MCP1703CB, U1 MICRO-USB-SHIELD-ZX62R-B-5P

Commit message: Eagle: - Risa zdroj - Kovanda termoclanky - Quanti akcelerometr
Other:
- board text added: "C1"
- board text added: "C2"
- board text added: "C3"
- board text added: "C4"
- board text added: "C5"
- board text added: "IC1"
- board text added: "IO1"
- board text added: "LED1"
- board text added: "R1"
- board text added: "R2"
- board text added: "R3"
- board text added: "R4"
- board text added: "R5"
- board text added: "R6"
- board text added: "R7"
- board text added: "R8"
- board text added: "U1"
Changed lines of the file:
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@@
 <layer number="25" name="tNames" color="7" fill="1" visible="yes" active="yes"/>
 <layer number="26" name="bNames" color="7" fill="1" visible="yes" active="yes"/>
-<layer number="27" name="tValues" color="7" fill="1" visible="no" active="yes"/>
+<layer number="27" name="tValues" color="7" fill="1" visible="yes" active="yes"/>
 <layer number="28" name="bValues" color="7" fill="1" visible="yes" active="yes"/>
 <layer number="29" name="tStop" color="7" fill="3" visible="yes" active="yes"/>
-<layer number="30" name="bStop" color="7" fill="6" visible="no" active="yes"/>
-<layer number="31" name="tCream" color="7" fill="4" visible="no" active="yes"/>
-<layer number="32" name="bCream" color="7" fill="5" visible="no" active="yes"/>
-<layer number="33" name="tFinish" color="6" fill="3" visible="no" active="yes"/>
-<layer number="34" name="bFinish" color="6" fill="6" visible="no" active="yes"/>
-<layer number="35" name="tGlue" color="7" fill="4" visible="no" active="yes"/>
-<layer number="36" name="bGlue" color="7" fill="5" visible="no" active="yes"/>
-<layer number="37" name="tTest" color="7" fill="1" visible="no" active="yes"/>
-<layer number="38" name="bTest" color="7" fill="1" visible="no" active="yes"/>
+<layer number="30" name="bStop" color="7" fill="6" visible="yes" active="yes"/>
+<layer number="31" name="tCream" color="7" fill="4" visible="yes" active="yes"/>
+<layer number="32" name="bCream" color="7" fill="5" visible="yes" active="yes"/>
+<layer number="33" name="tFinish" color="6" fill="3" visible="yes" active="yes"/>
+<layer number="34" name="bFinish" color="6" fill="6" visible="yes" active="yes"/>
+<layer number="35" name="tGlue" color="7" fill="4" visible="yes" active="yes"/>
+<layer number="36" name="bGlue" color="7" fill="5" visible="yes" active="yes"/>
+<layer number="37" name="tTest" color="7" fill="1" visible="yes" active="yes"/>
+<layer number="38" name="bTest" color="7" fill="1" visible="yes" active="yes"/>
 <layer number="39" name="tKeepout" color="4" fill="11" visible="yes" active="yes"/>
 <layer number="40" name="bKeepout" color="1" fill="11" visible="yes" active="yes"/>
@@
 <layer number="42" name="bRestrict" color="1" fill="10" visible="yes" active="yes"/>
 <layer number="43" name="vRestrict" color="2" fill="10" visible="yes" active="yes"/>
-<layer number="44" name="Drills" color="7" fill="1" visible="no" active="yes"/>
-<layer number="45" name="Holes" color="7" fill="1" visible="no" active="yes"/>
-<layer number="46" name="Milling" color="3" fill="1" visible="no" active="yes"/>
-<layer number="47" name="Measures" color="7" fill="1" visible="no" active="yes"/>
+<layer number="44" name="Drills" color="7" fill="1" visible="yes" active="yes"/>
+<layer number="45" name="Holes" color="7" fill="1" visible="yes" active="yes"/>
+<layer number="46" name="Milling" color="3" fill="1" visible="yes" active="yes"/>
+<layer number="47" name="Measures" color="7" fill="1" visible="yes" active="yes"/>
 <layer number="48" name="Document" color="7" fill="1" visible="yes" active="yes"/>
 <layer number="49" name="Reference" color="7" fill="1" visible="yes" active="yes"/>
@@
 <layer number="121" name="_tsilk" color="7" fill="1" visible="yes" active="yes"/>
 <layer number="122" name="_bsilk" color="7" fill="1" visible="yes" active="yes"/>
+<layer number="125" name="_tNames" color="14" fill="1" visible="yes" active="yes"/>
 <layer number="151" name="HeatSink" color="7" fill="1" visible="yes" active="yes"/>
 <layer number="200" name="200bmp" color="1" fill="10" visible="yes" active="yes"/>
@@
 <wire x1="35.54" y1="30.15" x2="0" y2="30.15" width="0" layer="20"/>
 <wire x1="0" y1="30.15" x2="0" y2="0" width="0" layer="20"/>
+<text x="9.525" y="12.065" size="1.27" layer="125">C1</text>
+<text x="14.605" y="4.445" size="1.27" layer="125" rot="R180">C2</text>
+<text x="27.305" y="14.605" size="1.27" layer="125">C3</text>
+<text x="27.305" y="18.415" size="1.27" layer="125">C4</text>
+<text x="21.59" y="25.4" size="1.27" layer="125" rot="R180">C5</text>
+<text x="13.335" y="12.065" size="1.27" layer="125">IC1</text>
+<text x="19.304" y="15.494" size="1.27" layer="125" rot="R90">IO1</text>
+<text x="23.859996875" y="2.810003125" size="1.27" layer="125" rot="R180">LED1</text>
+<text x="24.765" y="8.255" size="1.27" layer="125" rot="R270">R1</text>
+<text x="24.13" y="24.13" size="1.27" layer="125" rot="R180">R2</text>
+<text x="13.97" y="22.86" size="1.27" layer="125" rot="R180">R3</text>
+<text x="10.795" y="22.86" size="1.27" layer="125" rot="R180">R4</text>
+<text x="18.415" y="23.495" size="1.27" layer="125" rot="R180">R5</text>
+<text x="21.59" y="8.255" size="1.27" layer="125" rot="R270">R6</text>
+<text x="19.685" y="13.335" size="1.27" layer="125" rot="R180">R7</text>
+<text x="17.145" y="3.81" size="1.27" layer="125" rot="R90">R8</text>
+<text x="9.525" y="15.24" size="1.27" layer="125" rot="R180">U1</text>
 </plain>
 <attributes>
