File: EagleGit/quanti/ICM20600.brd (EAGLE design)
At the start: 35.5 x 30.1 mm, 21 parts, among them IC1 MCP1703CB, U1 MICRO-USB-SHIELD-ZX62R-B-5P

Commit message: Eagle: - Risa zdroj - Kovanda termoclanky - Quanti akcelerometr
Parts:
- IO1: value (none) -> ICM2600
Changed lines of the file:
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@@
 <attribute name="VALUE" x="12.065" y="6.35" size="1.27" layer="27"/>
 </element>
-<element name="IO1" library="gyro" package="LGA14" value="" x="21.59" y="15.494" smashed="yes" rot="R90">
+<element name="IO1" library="gyro" package="LGA14" value="ICM2600" x="21.59" y="15.494" smashed="yes" rot="R90">
 <attribute name="VALUE" x="16.51" y="15.494" size="1.27" layer="27" rot="R90"/>
 <attribute name="NAME" x="19.304" y="15.494" size="1.27" layer="25" rot="R90"/>
