File: EagleGit/quanti/ICM20600.sch (EAGLE design)
At the start: 21 parts, among them IC1 MCP1703CB, U1 MICRO-USB-SHIELD-ZX62R-B-5P

Commit message: Eagle: - Risa zdroj - Kovanda termoclanky - Quanti akcelerometr
Parts:
- IO1: value (none) -> ICM2600
Changed lines of the file:
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@@
 </classes>
 <parts>
-<part name="IO1" library="gyro" deviceset="ICM20600" device=""/>
+<part name="IO1" library="gyro" deviceset="ICM20600" device="" value="ICM2600"/>
 <part name="U1" library="con-hirose" deviceset="MICRO-USB-SHIELD-" device="ZX62R-B-5P"/>
 <part name="H1" library="holes" deviceset="MOUNT-PAD-ROUND" device="3.2"/>
