File: EagleGit/quanti/MOD1600.sch (EAGLE design)
At the start: 15 parts, among them IC1 MCP1703CB

Commit message: Eagle: - Risa zdroj - Kovanda termoclanky - Quanti akcelerometr
Other:
- moved on the sheet: JP1, LED1, R8
