File: EagleGit/quanti/PANEL.brd (EAGLE design)
At the start: 0 parts

Commit message: Eagle: - Risa zdroj - Kovanda termoclanky - Quanti akcelerometr
Parts:
- added C1, C11, C12, C2, C6, C7: 2u2, rcl:C0603
- added C10, C13, C14, C15, C3, C4, C5, C8, C9: 100n, rcl:C0603
- added H1, H10, H11, H12, H2, H3, H4, H5, H6, H7, H8, H9: MOUNT-PAD-ROUND3.2, holes:3,2-PAD
- added IC1, IC2, IC3: MCP1703CB, linear:SOT23
- added IO1: (no value), gyro:LGA14
- added IO2: (no value), gyro:LGA16
- added IO3: (no value), gyro:LGA_MOD1600
- added JP1: (no value), pinhead:1X07/90
- added LED1, LED2, LED3: (no value), led:SML0603
- added OSC1: KC2520B32K7680CM2E00, gyro:SMD_OSC
- added R1, R10, R11, R12, R13, R2, R3, R4, R5, R6, R9: 10k, rcl:R0603
- added R14, R7: 0R, rcl:R0603
- added R15, R16, R8: 220R, rcl:R0603
- added U1: MICRO-USB-SHIELD-ZX62R-B-5P, con-hirose:ZX62R-B-5P
- added U2: MICRO-USB, con-hirose:ZX62R-B-5P
Connections:
- new net +3V1: C7.1, C8.1, C9.1, IC2.2, IO2.P1, IO2.P16, R10.2, R11.2, R12.2, R13.2, R15.2, R9.2
- new net +3V2: C12.1, C13.1, C14.1, IC3.2, IO3.P1, OSC1.4, R16.2
- new net +3V3: C2.1, C3.1, C4.1, IC1.2, IO1.P5, IO1.P8, R1.2, R2.2, R3.2, R4.2, R5.2, R6.2, R8.2
- new net +5V: C1.1, IC1.3, U1.1
- new net +5V1: C6.1, IC2.3, U2.1
- new net +5V2: C11.1, C15.1, IC3.3, IO3.P15, JP1.7
- new net CLKIN: IO3.P6, OSC1.3
- new net DRDY: IO3.P10, JP1.2
- new net GND: C1.2, C2.2, C3.2, C4.2, C5.2, H1.B3,2, H2.B3,2, H3.B3,2, H4.B3,2, IC1.1, IO1.P10, IO1.P6, IO1.P7, LED1.C, R7.1, U1.5, U1.M1, U1.M2, U1.M3, U1.M4
- new net GND1: C10.2, C6.2, C7.2, C8.2, C9.2, H5.B3,2, H6.B3,2, H7.B3,2, H8.B3,2, IC2.1, IO2.P10, IO2.P11, IO2.P12, IO2.P13, IO2.P15, IO2.P8, IO2.P9, LED2.C, R14.1, U2.5, U2.M1, U2.M2, U2.M3, U2.M4
- new net GND2: C11.2, C12.2, C13.2, C14.2, C15.2, H10.B3,2, H11.B3,2, H12.B3,2, H9.B3,2, IC3.1, IO3.P13, IO3.P9, JP1.1, LED3.C, OSC1.2
- new net N$1: IO1.P9, R2.1
- new net N$10: C10.1, IO2.P14
- new net N$11: IO2.P2, R10.1, U2.2
- new net N$12: IO2.P3, R9.1, U2.3
- new net N$13: IO2.P5, R11.1
- new net N$14: IO2.P4, R12.1, R14.2
- new net N$15: IO2.P6, R13.1
- new net N$16: LED3.A, R16.1
- new net N$2: IO1.P4, R1.1
- new net N$3: C5.1, IO1.P11
- new net N$4: IO1.P13, R3.1, U1.2
- new net N$5: IO1.P14, R4.1, U1.3
- new net N$6: LED2.A, R15.1
- new net N$7: IO1.P12, R5.1
- new net N$8: IO1.P1, R6.1, R7.2
- new net N$9: LED1.A, R8.1
- new net NCS: IO3.P2, JP1.6
- new net SCLK: IO3.P5, JP1.3
- new net SDI: IO3.P4, JP1.4
- new net SDO: IO3.P3, JP1.5
Routing:
- net +3V1: track 0.00 -> 67.2 mm
- net +3V3: track 0.00 -> 65.0 mm
- net GND1: track 0.00 -> 55.3 mm, vias 0 -> 9
- net GND: track 0.00 -> 48.7 mm, vias 0 -> 8
- net +3V2: track 0.00 -> 47.9 mm, vias 0 -> 2
- net +5V2: track 0.00 -> 40.0 mm
- net GND2: track 0.00 -> 35.9 mm, vias 0 -> 5
- net DRDY: track 0.00 -> 26.6 mm, vias 0 -> 2
- net N$4: track 0.00 -> 20.3 mm, vias 0 -> 2
- net N$11: track 0.00 -> 20.2 mm, vias 0 -> 2
- net N$5: track 0.00 -> 19.3 mm
- net N$12: track 0.00 -> 16.8 mm
- net NCS: track 0.00 -> 15.0 mm
- net SDO: track 0.00 -> 14.8 mm
- net SDI: track 0.00 -> 14.6 mm
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- added copper zone on layer 16, net GND
- added copper zone on layer 16, net GND1
- added copper zone on layer 16, net GND2
Other:
- board outline added: 80 x 69.5 mm
- board text added: "C1"
- board text added: "C2"
- board text added: "C3"
- board text added: "C4"
- board text added: "C5"
- board text added: "IC1"
- board text added: "IO1"
- board text added: "JP1"
- board text added: "LED1"
- board text added: "OSC1"
- board text added: "R1"
- board text added: "R2"
- board text added: "R3"
- board text added: "R4"
- board text added: "R5"
- board text added: "R6"
- board text added: "R7"
- board text added: "R8"
- board text added: "U1"
